File: PCB/beat_sensing_ledHat/beat_sensing_ledHat.kicad_sch (KiCad schematic)
At the start: 0 parts

Commit message: PCB Designing
Parts:
- added C1, C2, C3, C4, C5: 10n, Capacitor_THT:C_Disc_D8.0mm_W2.5mm_P5.00mm, symbol Device:C
- added J1: LM324, Package_DIP:DIP-14_W7.62mm_Socket, symbol IC_14_HOLDER:1-2199298-3
- added J2: Screw_Terminal_01x02, TerminalBlock:TerminalBlock_MaiXu_MX126-5.0-02P_1x02_P5.00mm, symbol Connector:Screw_Terminal_01x02
- added J3: Microphone, Connector_PinHeader_2.54mm:PinHeader_1x03_P2.54mm_Vertical, symbol Connector:Conn_01x03_Pin
- added J4: LED, Connector_PinHeader_2.54mm:PinHeader_1x03_P2.54mm_Vertical, symbol Connector:Conn_01x03_Pin
- added R1, R10, R9: 4.7k, Resistor_THT:R_Axial_DIN0207_L6.3mm_D2.5mm_P10.16mm_Horizontal, symbol Device:R
- added R2, R8: 10k, Resistor_THT:R_Axial_DIN0207_L6.3mm_D2.5mm_P10.16mm_Horizontal, symbol Device:R
- added R3, R4: 2.2k, Resistor_THT:R_Axial_DIN0411_L9.9mm_D3.6mm_P15.24mm_Horizontal, symbol Device:R
- added R5, R6: 75k, Resistor_THT:R_Axial_DIN0207_L6.3mm_D2.5mm_P10.16mm_Horizontal, symbol Device:R
- added R7: 5.6k, Resistor_THT:R_Axial_DIN0207_L6.3mm_D2.5mm_P10.16mm_Horizontal, symbol Device:R
- added U1: ARDUINO_NANO, nano:MODULE_ARDUINO_NANO, symbol ARDUINO_NANO:ARDUINO_NANO
Connections:
- new net: C3.1, J3.3 (Pin_3), R10.1
- new net: C1.1, C2.1, C3.2, R3.2
- new net: C1.2, C2.2, J1.3, R4.2
- new net: J1.13, R7.1, R8.2
- new net: C4.2, J1.12, R9.2
- new net: J1.2, R1.1, R2.2
- new net: C5.2, R10.2, R9.1
- new net: U1.28 (RESET), U1.3 (RESET)
- new net: J4.2 (Pin_2), U1.6 (D3)
- new net 1.65V: R2.1, R4.1, R5.2, R6.1
- new net GND: C4.1, J1.11, J2.2 (Pin_2), J3.2 (Pin_2), J4.3 (Pin_3), R5.1, R8.1, U1.29 (GND_29)
- new net HP: J1.1, R1.2, R3.1, U1.19 (A0)
- new net LP: C5.1, J1.14, R7.2, U1.25 (A6)
- new net VBATT: J1.4, J2.1 (Pin_1), J3.1 (Pin_1), J4.1 (Pin_1), R6.2, U1.27 (+5V)
- no-connect marks 0 -> 30
